File: obc-ssm.sch (KiCad schematic (older format))
At the start: 0 parts

Commit message: obc updated
Parts:
- added C? (x3): C, symbol C
- added C? (x2): 22pF, symbol C_Small
- added C?: C_Small, symbol C_Small
- added OBC_32MI: ATMEGA32M1-MU, QFN32, symbol ATMEGA32M1-MU
- added R? (x2): R, symbol R
- added U?: SN65HVD230, Housings_SOIC:SOIC-8_3.9x4.9mm_Pitch1.27mm, symbol SN65HVD230
- added Y1: 8MHz, symbol Crystal_GND24
- added Y?: Crystal_GND23, symbol Crystal_GND23
Connections:
- new net +3V3: C?.2, OBC_32MI.19 (AVCC), OBC_32MI.21 (AREF(ISRC)), OBC_32MI.4 (VCC), U?.3 (VCC)
- new net CANH: R?.1, U?.7 (CANH)
- new net CANL: R?.2, U?.6 (CANL)
- new net CAN_LPWR: OBC_32MI.23 ((PCINT3/AMP0-)PB3), U?.8 (Rs)
- new net COM_RST: OBC_32MI.22 ((PCINT14/ADC10/ACMP1)PC6)
- new net EPS_RST: OBC_32MI.18 ((PCINT13/ADC9/ACMP3/AMP1+)PC5)
- new net GND: C?.1, C?.1, C?.1, C?.2, OBC_32MI.10 ((PCINT25/OC0B/XTAL1)PE1), OBC_32MI.11 ((PCINT26/ADC0/XTAL2)PE2), OBC_32MI.20 (AGND), OBC_32MI.5 (GND), R?.2, U?.2 (GND), Y1.2, Y1.4
- new net LOPWR: OBC_32MI.16 ((PCINT2/ADC5/INT1/ACMPN0)PB2)
- new net MISO: OBC_32MI.8 ((PCINT0/MISO/PSCOUT2A)PB0)
- new net MOSI: OBC_32MI.9 ((PCINT1/MOSI/PSCOUT2B)PB1)
- new net OBC_CAN_RX: OBC_32MI.7 ((PCINT11/T1/ICP1B/RXCAN)PC3)
- new net OBC_CAN_TX: OBC_32MI.6 ((PCINT10/T0/TXCAN)PC2)
- new net OBC_MISO_A: OBC_32MI.1 ((PCINT18/PSCIN2/OC1A/MISO_A)PD2)
- new net OBC_MOSI_A: OBC_32MI.2 ((PCINT19/TXD/TXLIN/OC0A/~SS~/MOSI_A)PD3)
- new net OBC_RST: OBC_32MI.17 ((PCINT12/ADC8/ACMPN3/AMP1-)PC4)
- new net OBC_SCK_A: OBC_32MI.12 ((PCINT20/ADC1/RXD/RXLIN/ICP1A/SCK_A)PD4)
- new net PAY_RST: OBC_32MI.25 ((PCINT15/D2A/AMP2+)PC7)
- new net SCK: OBC_32MI.28 ((PCINT7/ADC4/SCK/PSCOUT0B)PB7)
- no-connect marks 0 -> 11
