File: com-ssm.sch (KiCad schematic (older format))
At the start: 11 parts

Commit message: almost done com subsheet
Parts:
- added C? (x3): 0.1uF, symbol C
- added D?: PWR_LED, symbol LED
- added J?: PROGRAMMING PORT, symbol Conn_02x03_Odd_Even
- added R?: 10K, symbol R
- added R?: 120R, symbol R
- SW?: value SW_Push_Dual -> COM_SW_RST
Connections:
- net +3V3: now also U?.19 (AVCC), U?.21 (AREF(ISRC)), U?.4 (VCC), C?.2, C?.2, C?.2, J?.2 (Pin_2), R?.1, R?.1
- net COM_MISO_A: now also J?.1 (Pin_1)
- net COM_MOSI_A: now also J?.4 (Pin_4)
- net COM_RST: now also SW?.1, SW?.3, J?.5 (Pin_5), R?.2
- net COM_SCK_A: now also J?.3 (Pin_3)
- net GND: now also SW?.2, SW?.4, C?.1, C?.1, C?.1, D?.1 (K), J?.6 (Pin_6)
- new net: D?.2 (A), R?.2
Other:
- note added: "PINS YOU NEED TO HAVE COME IN:\n* 9VCRIT\n*3V3CRIT\n*CANH\n*CANL\n\n\nPINS YOU NEED TO HAVE GO OUT:\n*OBC_RST\n*"
- note removed: "add power bit"
- note removed: "add programming port"
- note removed: "finish this"
- moved on the sheet: C?, L?, R?, SW?, U?, Y?
